File: main_module.brd (EAGLE design)
At the start: 70.2 x 100.3 mm, 64 parts, among them CN1 SWD, CN2 USB, IC1 STM32F103C8T, IC2 TP4056, IC3 MCP1700T-3302E, Q1 32768, Q2 8MHz

Commit message: improvements
Parts:
- added JP9: +V_BATERY, adafruit:1X1-BIGPOGO
- JP7: value +VBAT -> +VBAT_SWITCH
- moved R7 0.76 mm to (45.2, 7.62)
Connections:
- new net +V_BATTERY: IC2.5, JP9.P$1
- net V+: no longer IC2.5
Routing:
- net +V_BATTERY: track 0.00 -> 14.3 mm
- net V+: track 96.7 -> 91.2 mm
Changed lines of the file:
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@@
 <element name="JP4" library="adafruit" package="1X1-BIGPOGO" value="SBM+" x="3.81" y="2.54" rot="R180"/>
 <element name="JP6" library="adafruit" package="1X1-BIGPOGO" value="SBM-" x="3.81" y="97.79" rot="R180"/>
-<element name="JP7" library="adafruit" package="1X1-BIGPOGO" value="+VBAT" x="33.02" y="4.318" rot="R90"/>
+<element name="JP7" library="adafruit" package="1X1-BIGPOGO" value="+VBAT_SWITCH" x="33.02" y="4.318" rot="R90"/>
 <element name="JP8" library="adafruit" package="1X1-BIGPOGO" value="GND" x="29.21" y="4.318" rot="R90"/>
 <element name="R12" library="resistor" package="M0805" value="4.7M" x="4.445" y="14.224" rot="R270"/>
@@
 <element name="R9" library="resistor" package="M0805" value="2k" x="50.8" y="3.81" rot="R180"/>
 <element name="LED1" library="led" package="CHIP-LED0805" value="CHARGE" x="45.72" y="5.08" rot="R90"/>
-<element name="R7" library="resistor" package="M0805" value="1k" x="44.45" y="7.62"/>
+<element name="R7" library="resistor" package="M0805" value="1k" x="45.212" y="7.62"/>
 <element name="C10" library="resistor" package="C0805" value="10uF" x="54.61" y="3.81" rot="R180"/>
 <element name="JP1" library="adafruit" package="1X1-BIGPOGO" value="+VBCK_BAT" x="67.31" y="62.23" rot="R180"/>
@@
 <element name="R20" library="resistor" package="M0805" value="150" x="18.796" y="63.881" rot="R180"/>
 <element name="R21" library="resistor" package="M0805" value="270k" x="6.35" y="44.45" rot="R180"/>
+<element name="JP9" library="adafruit" package="1X1-BIGPOGO" value="+V_BATERY" x="39.37" y="2.54"/>
 </elements>
 <signals>
@@
 <contactref element="R4" pad="2"/>
 <contactref element="IC3" pad="3"/>
-<contactref element="IC2" pad="5"/>
 <wire x1="32.9184" y1="4.3434" x2="33.02" y2="4.318" width="0.508" layer="16"/>
 <wire x1="33.0327" y1="4.3434" x2="33.02" y2="4.318" width="0.508" layer="1"/>
@@
 <wire x1="31.75" y1="8.89" x2="33.02" y2="7.62" width="1.016" layer="16"/>
 <wire x1="33.02" y1="7.62" x2="33.02" y2="4.318" width="1.016" layer="16"/>
-<wire x1="48.05" y1="10.795" x2="42.515" y2="10.795" width="0.8128" layer="1"/>
-<wire x1="42.515" y1="10.795" x2="41.895" y2="11.415" width="0.8128" layer="1"/>
+<wire x1="41.245" y1="10.795" x2="41.895" y2="11.415" width="0.8128" layer="1"/>
 </signal>
 <signal name="HV_PULSE">
@@
 <contactref element="R7" pad="2"/>
 <wire x1="46.0629" y1="8.2296" x2="48.006" y2="8.2296" width="0.6096" layer="1"/>
-<wire x1="45.4914" y1="7.6581" x2="46.0629" y2="8.2296" width="0.254" layer="1"/>
+<wire x1="46.1264" y1="7.9121" x2="46.0629" y2="8.2296" width="0.254" layer="1"/>
 <wire x1="48.006" y1="8.2296" x2="48.05" y2="8.255" width="0.254" layer="1"/>
-<wire x1="45.4914" y1="7.6581" x2="45.4" y2="7.62" width="0.254" layer="1"/>
+<wire x1="46.1264" y1="7.9121" x2="46.162" y2="7.62" width="0.254" layer="1"/>
 </signal>
 <signal name="N$25">
@@
 <contactref element="LED1" pad="C"/>
 <wire x1="44.67" y1="5.08" x2="44.45" y2="5.08" width="0.3048" layer="1"/>
-<wire x1="44.45" y1="5.08" x2="43.18" y2="6.35" width="0.6096" layer="1"/>
-<wire x1="43.18" y1="6.35" x2="43.18" y2="7.3" width="0.6096" layer="1"/>
-<wire x1="43.18" y1="7.3" x2="43.5" y2="7.62" width="0.3048" layer="1"/>
+<wire x1="44.45" y1="5.08" x2="44.069" y2="6.731" width="0.6096" layer="1"/>
+<wire x1="44.069" y1="6.731" x2="44.069" y2="7.554" width="0.6096" layer="1"/>
+<wire x1="44.069" y1="7.554" x2="44.262" y2="7.62" width="0.3048" layer="1"/>
 </signal>
 <signal name="+VBCK_BAT">
@@
 <wire x1="15.5702" y1="63.881" x2="12.1412" y2="67.31" width="0.6096" layer="1"/>
 </signal>
+<signal name="+V_BATTERY">
+<contactref element="IC2" pad="5"/>
+<contactref element="JP9" pad="P$1"/>
+<wire x1="48.05" y1="10.795" x2="43.815" y2="10.795" width="1.016" layer="1"/>
+<wire x1="43.815" y1="10.795" x2="41.91" y2="8.89" width="1.016" layer="1"/>
+<wire x1="41.91" y1="8.89" x2="41.91" y2="7.62" width="1.016" layer="1"/>
+<wire x1="41.91" y1="7.62" x2="40.64" y2="6.35" width="1.016" layer="1"/>
+<wire x1="40.64" y1="6.35" x2="40.64" y2="3.81" width="1.016" layer="1"/>
+<wire x1="40.64" y1="3.81" x2="39.37" y2="2.54" width="1.016" layer="1"/>
+</signal>
 </signals>
